Commit message: bot arranged

File: src/description/bot.urdf.xacro (robot description, xacro)
@@ -1,4 +1,4 @@
 <robot xmlns:xacro="http://www.ros.org/wiki/xacro">
-	<!-- <xacro:include filename="wheel.urdf.xacro" /> -->
+	<xacro:include filename="wheel.urdf.xacro" />
 	<joint name="base_joint" type="fixed">
 		<parent link="base_link" />
@@ -9,5 +9,5 @@
 	<link name="bot_base">
 		<visual>
-			<origin xyz="0.056 0.0 0.025" rpy="0.0 0.0 ${pi}" />
+			<origin xyz="0.0615 0.0 0.025" rpy="0.0 0.0 ${pi}" />
 			<geometry>
 				<!-- <box size="0.3 0.2 0.1" /> -->
@@ -19,5 +19,5 @@
 		</visual>
 		<collision>
-			<origin xyz="0.075 0.0 0.025" />
+			<origin xyz="0.0615 0.0 0.025" rpy="0.0 0.0 ${pi}" />
 			<geometry>
 				<!-- <box size="0.3 0.2 0.1" /> -->
@@ -26,15 +26,15 @@
 		</collision>
 	</link>
-	<!-- <xacro:wheel suffix="left" parent="bot_base">
-		<origin xyz="0.0 -0.125 0.0" rpy="${pi/2} 0.0 0.0 " />
+	<xacro:wheel suffix="left" parent="bot_base">
+		<origin xyz="0.0 -0.083 0.046" rpy="0.0 0.0 0.0 " />
 	</xacro:wheel>
 	<xacro:wheel suffix="right" parent="bot_base">
-		<origin xyz="0.0 0.125 0.0" rpy="${pi/2} 0.0 0.0" />
-	</xacro:wheel> -->
+		<origin xyz="0.0 0.083 0.046" rpy="${pi} 0.0 0.0" />
+	</xacro:wheel>
 	<joint name="castor_joint" type="fixed">
 		<parent link="bot_base" />
 		<child link="castor_wheel" />
 		<axis xyz="0.0 0.0 0.0" />
-		<origin xyz="0.130 0.0 0.0075" rpy="0.0 0.0 0.0" />
+		<origin xyz="0.135 0.0 0.0075" rpy="0.0 0.0 0.0" />
 	</joint>
 	<link name="castor_wheel">

File: src/description/wheel.urdf.xacro (robot description, xacro)
@@ -11,5 +11,5 @@
 				<geometry>
 					<!-- <cylinder radius="0.05" length="0.05" /> -->
-                    <mesh filename="description/meshes/Wheel.stl" />
+                    <mesh filename="package://diff_bot/description/meshes/Wheel.stl" />
 				</geometry>
 				<material name="red">
@@ -20,5 +20,5 @@
 				<geometry>
 					<!-- <cylinder radius="0.05" length="0.05" /> -->
-                    <mesh filename="description/meshes/Wheel.stl" />
+                    <mesh filename="package://diff_bot/description/meshes/Wheel.stl" />
 				</geometry>
 			</collision>
